File: kicad_source/imu.sch (KiCad schematic (older format))
At the start: 1 part, among them U6 BNO085

Commit message: added BMP388
Parts:
- added C1, C2: 100nF, capacitors:C_0603, symbol devices:C_0603
- added U7: BMP388, IC_sensor:BMP388, symbol IC_sensor:BMP388
Connections:
- net labels added: BMP388_INT
- wire segments 10 -> 30
Changed lines of the file:
@@
 Text Label 2100 3650 0    50   ~ 0
 I2C_SCL
+$Comp
+L IC_sensor:BMP388 U7
+U 1 1 5ED82558
+P 7750 3100
+F 0 "U7" H 7750 3525 50  0000 C CNN
+F 1 "BMP388" H 7750 3434 50  0000 C CNN
+F 2 "IC_sensor:BMP388" H 7750 3100 50  0001 C CNN
+F 3 "" H 7750 3100 50  0001 C CNN
+	1    7750 3100
+	1    0    0    -1
+$EndComp
+$Comp
+L devices:C_0603 C1
+U 1 1 5ED83121
+P 8300 3100
+F 0 "C1" H 8392 3146 50  0000 L CNN
+F 1 "100nF" H 8392 3055 50  0000 L CNN
+F 2 "capacitors:C_0603" H 8300 2950 50  0001 C CNN
+F 3 "" H 8300 3100 50  0000 C CNN
+	1    8300 3100
+	1    0    0    -1
+$EndComp
+$Comp
+L devices:C_0603 C2
+U 1 1 5ED83CAD
+P 8750 3100
+F 0 "C2" H 8842 3146 50  0000 L CNN
+F 1 "100nF" H 8842 3055 50  0000 L CNN
+F 2 "capacitors:C_0603" H 8750 2950 50  0001 C CNN
+F 3 "" H 8750 3100 50  0000 C CNN
+	1    8750 3100
+	1    0    0    -1
+$EndComp
+$Comp
+L power-supply:+3.3V #PWR018
+U 1 1 5ED842B7
+P 8300 2800
+F 0 "#PWR018" H 8300 2650 50  0001 C CNN
+F 1 "+3.3V" H 8315 2973 50  0000 C CNN
+F 2 "" H 8300 2800 50  0000 C CNN
+F 3 "" H 8300 2800 50  0000 C CNN
+	1    8300 2800
+	1    0    0    -1
+$EndComp
+$Comp
+L power-supply:+3.3V #PWR020
+U 1 1 5ED84CFF
+P 8750 2800
+F 0 "#PWR020" H 8750 2650 50  0001 C CNN
+F 1 "+3.3V" H 8765 2973 50  0000 C CNN
+F 2 "" H 8750 2800 50  0000 C CNN
+F 3 "" H 8750 2800 50  0000 C CNN
+	1    8750 2800
+	1    0    0    -1
+$EndComp
+$Comp
+L power-supply:GND #PWR017
+U 1 1 5ED8524F
+P 8150 3350
+F 0 "#PWR017" H 8150 3100 50  0001 C CNN
+F 1 "GND" H 8155 3177 50  0000 C CNN
+F 2 "" H 8150 3350 50  0000 C CNN
+F 3 "" H 8150 3350 50  0000 C CNN
+	1    8150 3350
+	1    0    0    -1
+$EndComp
+$Comp
+L power-supply:GND #PWR019
+U 1 1 5ED8591C
+P 8300 3250
+F 0 "#PWR019" H 8300 3000 50  0001 C CNN
+F 1 "GND" H 8305 3077 50  0000 C CNN
+F 2 "" H 8300 3250 50  0000 C CNN
+F 3 "" H 8300 3250 50  0000 C CNN
+	1    8300 3250
+	1    0    0    -1
+$EndComp
+$Comp
+L power-supply:GND #PWR021
+U 1 1 5ED85A93
+P 8750 3250
+F 0 "#PWR021" H 8750 3000 50  0001 C CNN
+F 1 "GND" H 8755 3077 50  0000 C CNN
+F 2 "" H 8750 3250 50  0000 C CNN
+F 3 "" H 8750 3250 50  0000 C CNN
+	1    8750 3250
+	1    0    0    -1
+$EndComp
+Wire Wire Line
+	8100 3100 8150 3100
+Wire Wire Line
+	8150 3100 8150 3200
+Wire Wire Line
+	8300 3200 8300 3250
+Wire Wire Line
+	8750 3200 8750 3250
+Wire Wire Line
+	8300 2800 8300 3000
+Wire Wire Line
+	8750 2800 8750 2900
+Wire Wire Line
+	8100 3000 8300 3000
+Connection ~ 8300 3000
+Wire Wire Line
+	8100 2900 8750 2900
+Connection ~ 8750 2900
+Wire Wire Line
+	8750 2900 8750 3000
+Wire Wire Line
+	8100 3300 8150 3300
+Connection ~ 8150 3300
+Wire Wire Line
+	8150 3300 8150 3350
+Wire Wire Line
+	8100 3200 8150 3200
+Connection ~ 8150 3200
+Wire Wire Line
+	8150 3200 8150 3300
+$Comp
+L power-supply:GND #PWR016
+U 1 1 5ED8722B
+P 7350 3350
+F 0 "#PWR016" H 7350 3100 50  0001 C CNN
+F 1 "GND" H 7355 3177 50  0000 C CNN
+F 2 "" H 7350 3350 50  0000 C CNN
+F 3 "" H 7350 3350 50  0000 C CNN
+	1    7350 3350
+	1    0    0    -1
+$EndComp
+Wire Wire Line
+	7400 3000 7350 3000
+Wire Wire Line
+	7350 3000 7350 3350
+Wire Wire Line
+	6550 3300 7400 3300
+Wire Wire Line
+	6550 3100 7400 3100
+Wire Wire Line
+	6550 2900 7400 2900
+Text Label 6700 3100 0    50   ~ 0
+I2C_SCL
+Text Label 6700 2900 0    50   ~ 0
+I2C_SDA
+Text Label 6700 3300 0    50   ~ 0
+BMP388_INT
+$Comp
+L power-supply:+3.3V #PWR015
+U 1 1 5ED8AB19
+P 7250 2750
+F 0 "#PWR015" H 7250 2600 50  0001 C CNN
+F 1 "+3.3V" H 7265 2923 50  0000 C CNN
+F 2 "" H 7250 2750 50  0000 C CNN
+F 3 "" H 7250 2750 50  0000 C CNN
+	1    7250 2750
+	1    0    0    -1
+$EndComp
+Wire Wire Line
+	7250 2750 7250 3200
+Wire Wire Line
+	7250 3200 7400 3200
 $EndSCHEMATC
